Commit message: change urdf to use obj

File: urdf/assembly_simple.urdf (robot description, URDF)
Before this commit: robot assembly_simple, 13 links, 12 joints
Links:
- link base_link: geometry collision mesh filename=package://assembly_simple_description/meshes/base_link.obj scale=0.001 0.001 0.001; visual mesh filename=package://assembly_simple_description/meshes/base_link.obj scale=0.001 0.001 0.001

Commit message: use absolute path

File: urdf/assembly_simple.urdf (robot description, URDF)
Before this commit: robot assembly_simple, 13 links, 12 joints
Links:
- link assembly_simplyv3_backup_Component6_Mirror__Mirror__v1_1: geometry collision mesh filename=/assembly_simple_description/meshes/assembly_simplyv3_backu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 scale=0.001 0.001 0.001; visual mesh filename=/assembly_simple_description/meshes/assembly_simplyv3_backu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 scale=0.001 0.001 0.001
- link assembly_simplyv3_backup_Component6_Mirror___1__v1_1: geometry collision mesh filename=/assembly_simple_description/meshes/assembly_simplyv3_backu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 scale=0.001 0.001 0.001; visual mesh filename=/assembly_simple_description/meshes/assembly_simplyv3_backu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 scale=0.001 0.001 0.001
- link assembly_simplyv3_backup_Component6_Mirror__v1_1: geometry collision mesh filename=/assembly_simple_description/meshes/assembly_simplyv3_backu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 scale=0.001 0.001 0.001; visual mesh filename=/assembly_simple_description/meshes/assembly_simplyv3_backu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 scale=0.001 0.001 0.001
- link assembly_simplyv3_backup_Component6_v1_1: geometry collision mesh filename=/assembly_simple_description/meshes/assembly_simplyv3_backu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 scale=0.001 0.001 0.001; visual mesh filename=/assembly_simple_description/meshes/assembly_simplyv3_backu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 scale=0.001 0.001 0.001
- link assembly_simplyv3_backup_hip_L_simple_v2_Mirror__Mirror__v1_1: geometry collision mesh filename=/assembly_simple_description/meshes/assembly_simplyv3_backu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 scale=0.001 0.001 0.001; visual mesh filename=/assembly_simple_description/meshes/assembly_simplyv3_backu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 scale=0.001 0.001 0.001
- link assembly_simplyv3_backup_hip_L_simple_v2_Mirror___1__v1_1: geometry collision mesh filename=/assembly_simple_description/meshes/assembly_simplyv3_backu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 scale=0.001 0.001 0.001; visual mesh filename=/assembly_simple_description/meshes/assembly_simplyv3_backu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 scale=0.001 0.001 0.001
- link assembly_simplyv3_backup_hip_L_simple_v2_Mirror__v1_1: geometry collision mesh filename=/assembly_simple_description/meshes/assembly_simplyv3_backu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 scale=0.001 0.001 0.001; visual mesh filename=/assembly_simple_description/meshes/assembly_simplyv3_backu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 scale=0.001 0.001 0.001
- link assembly_simplyv3_backup_hip_L_simple_v2_v1_1: geometry collision mesh filename=/assembly_simple_description/meshes/assembly_simplyv3_backu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 scale=0.001 0.001 0.001; visual mesh filename=/assembly_simple_description/meshes/assembly_simplyv3_backu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 scale=0.001 0.001 0.001
- link assembly_simplyv3_backup_lowerleg_left_v2_Mirror__Mirror__v1_1: geometry collision mesh filename=/assembly_simple_description/meshes/assembly_simplyv3_backu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 scale=0.001 0.001 0.001; visual mesh filename=/assembly_simple_description/meshes/assembly_simplyv3_backu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 scale=0.001 0.001 0.001
- link assembly_simplyv3_backup_lowerleg_left_v2_Mirror___1__v1_1: geometry collision mesh filename=/assembly_simple_description/meshes/assembly_simplyv3_backu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 scale=0.001 0.001 0.001; visual mesh filename=/assembly_simple_description/meshes/assembly_simplyv3_backu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 scale=0.001 0.001 0.001
- link assembly_simplyv3_backup_lowerleg_left_v2_Mirror__v1_1: geometry collision mesh filename=/assembly_simple_description/meshes/assembly_simplyv3_backu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 scale=0.001 0.001 0.001; visual mesh filename=/assembly_simple_description/meshes/assembly_simplyv3_backu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 scale=0.001 0.001 0.001
- link assembly_simplyv3_backup_lowerleg_left_v2_v1_1: geometry collision mesh filename=/assembly_simple_description/meshes/assembly_simplyv3_backu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 scale=0.001 0.001 0.001; visual mesh filename=/assembly_simple_description/meshes/assembly_simplyv3_backu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 scale=0.001 0.001 0.001
- link base_link: geometry collision mesh filename=/assembly_simple_description/meshes/base_link.obj scale=0.001 0.001 0.001; visual mesh filename=/assembly_simple_description/meshes/base_link.obj scale=0.001 0.001 0.001
